Commit message: #21 outdoot sim planner configured+outdoor collector

File: sirius/urdf/sirius_description.urdf (robot description, URDF)
Before this commit: robot None, 1 links, 1 joints
Links:
- link GPS_link: geometry visual mesh filename=package://robot_simulation/models/rtk/model.dae

Commit message: #24 gps driver

File: sirius/urdf/sirius_description.urdf (robot description, URDF)
Before this commit: robot None, 1 links, 1 joints
Joints:
- joint GPS_joint: origin xyz=-0.45 0 1 rpy=0 0 0 -> xyz=-0.2 0 0.045 rpy=0 0 0

Commit message: #35 mounting stand urdf + keyboard collector

File: sirius/urdf/sirius_description.urdf (robot description, URDF)
Before this commit: robot None, 1 links, 1 joints
Links:
- added link left_side_stand_link; visual mesh filename=package://sirius/urdf/meshes/sidestands_v2.STL scale=0.001 0.001 0.001
- added link mid_stand_link; visual mesh filename=package://sirius/urdf/meshes/mid_square.STL scale=0.001 0.001 0.001
- added link right_side_stand_link; visual mesh filename=package://sirius/urdf/meshes/sidestands_v2.STL scale=0.001 0.001 0.001
Joints:
- added joint left_side_stand_joint: type fixed, parent right_side_stand_link, child left_side_stand_link, origin xyz=0. 0.53 0.0 rpy=0 0 0
- added joint mid_stand_joint: type fixed, parent right_side_stand_link, child mid_stand_link, origin xyz=0.0 -0.012 0.49 rpy=0 0 0
- added joint right_side_stand_joint: type fixed, parent top_plate_link, child right_side_stand_link, origin xyz=-0.1 -0.255 0.005 rpy=0 0 0
- joint GPS_joint: origin xyz=-0.2 0 0.045 rpy=0 0 0 -> xyz=0.0 0.1 0.155 rpy=0 0 0; parent top_plate_link -> mid_stand_link
